Commit message: add aula11_ex6

File: Parte11/psr_aula11_ex6_scara/urdf/scara.urdf (robot description, URDF)
Before this commit: robot scara, 1 links, 0 joints
Links:
- added link ee_link; visual cylinder length=0.8 radius=0.05
- added link link_1; visual box size=1.5 0.4 0.3
- added link link_1_auxiliary; visual cylinder length=0.3 radius=0.2
- added link link_2; visual box size=1.2 0.4 0.3
- added link link_2_auxiliary; visual cylinder length=0.3 radius=0.2
- added link link_2_auxiliary_2; visual cylinder length=0.3 radius=0.2
- link base_link: geometry visual cylinder length=0.3 radius=0.2
Joints:
- added joint base_link_to_link_1: type revolute, parent base_link, child link_1, origin xyz=0 0 0.3 rpy=0 0 0, axis 0 0 1, limit lower=-3.14 upper=3.14 effort=1000.0 velocity=0.5
- added joint link_1_to_link_1_auxiliary: type fixed, parent link_1, child link_1_auxiliary, origin xyz=0 0 0 rpy=0 0 0
- added joint link_1_to_link_2: type revolute, parent link_1, child link_2, origin xyz=1.5 0 0 rpy=0 0 0, axis 0 0 1, limit lower=-1.57 upper=1.57 effort=1000.0 velocity=0.5
- added joint link_2_auxiliary_2_to_ee_link: type prismatic, parent link_2_auxiliary_2, child ee_link, origin xyz=0 0 0 rpy=0 1.57 0, axis 1 0 0, limit lower=0.35 upper=0.6 effort=1000.0 velocity=0.5
- added joint link_2_to_link_2_auxiliary: type fixed, parent link_2, child link_2_auxiliary, origin xyz=0 0 0 rpy=0 0 0
- added joint link_2_to_link_2_auxiliary_2: type fixed, parent link_2, child link_2_auxiliary_2, origin xyz=1.2 0 0 rpy=0 0 0
