Commit message: Add part13

File: Parte12/robutler_description/urdf/robutler.gazebo.xacro (robot description, xacro)
@@ -5,5 +5,5 @@
   <xacro:arg name="imu_visual"    default="false"/>
   <gazebo reference="base_link">
-    <material>Gazebo/Red</material>
+    <material>Gazebo/FlatBlack</material>
   </gazebo>
   <gazebo reference="wheel_left_link">
@@ -15,5 +15,6 @@
     <maxVel>0.1</maxVel>
     <fdir1>1 0 0</fdir1>
-    <material>Gazebo/FlatBlack</material>
+        <!-- <material>Gazebo/FlatBlack</material> -->
+    <material>Gazebo/Red</material>
   </gazebo>
   <gazebo reference="wheel_right_link">
@@ -25,5 +26,6 @@
     <maxVel>0.1</maxVel>
     <fdir1>1 0 0</fdir1>
-    <material>Gazebo/FlatBlack</material>
+        <!-- <material>Gazebo/FlatBlack</material> -->
+    <material>Gazebo/Red</material>
   </gazebo>
   <gazebo reference="caster_back_right_link">
@@ -103,5 +105,5 @@
   </gazebo>
   <gazebo reference="base_scan">
-    <material>Gazebo/Blue</material>
+    <material>Gazebo/White</material>
     <sensor type="ray" name="lds_lfcd_sensor">
       <pose>0 0 0 0 0 0</pose>
@@ -202,3 +204,9 @@
     </sensor>
   </gazebo>
+  <gazebo reference="base_antena">
+    <material>Gazebo/FlatBlack</material>
+  </gazebo>
+  <gazebo reference="antena">
+    <material>Gazebo/Red</material>
+  </gazebo>
 </robot>

File: Parte12/robutler_description/urdf/robutler.urdf.xacro (robot description, xacro)
@@ -16,5 +16,5 @@
         <mesh filename="package://turtlebot3_description/meshes/bases/waffle_pi_base.stl" scale="0.001 0.001 0.001"/>
       </geometry>
-      <material name="orange"/>
+      <material name="light_black"/>
     </visual>
     <collision>
@@ -44,5 +44,5 @@
         <mesh filename="package://turtlebot3_description/meshes/wheels/left_tire.stl" scale="0.001 0.001 0.001"/>
       </geometry>
-      <material name="white"/>
+      <material name="red"/>
     </visual>
     <collision>
@@ -72,5 +72,5 @@
         <mesh filename="package://turtlebot3_description/meshes/wheels/right_tire.stl" scale="0.001 0.001 0.001"/>
       </geometry>
-      <material name="white"/>
+      <material name="red"/>
     </visual>
     <collision>
@@ -145,5 +145,6 @@
         <mesh filename="package://turtlebot3_description/meshes/sensors/lds.stl" scale="0.001 0.001 0.001"/>
       </geometry>
-      <material name="dark"/>
+      <!-- <material name="dark"/> -->
+      <material name="white"/>
     </visual>
     <collision>
@@ -221,5 +222,6 @@
   <link name="base_antena">
     <visual>
-      <origin xyz="0 0 0.0725" rpy="0 0 0"/>
+      <!-- <origin xyz="0 0 0.0725" rpy="0 0 0"/> -->
+      <origin xyz="0 0 0.047" rpy="0 0 0"/>
       <geometry>
         <cylinder length="0.10" radius="0.003"/>
@@ -231,5 +233,5 @@
     <parent link="base_antena"/>
     <child link="antena"/>
-    <origin xyz="0 0 0.125" rpy="0 0 0"/>
+    <origin xyz="0 0 0.105" rpy="0 0 0"/>
   </joint>
   <link name="antena">
@@ -239,5 +241,5 @@
         <cylinder length="0.02" radius="0.030"/>
       </geometry>
-      <material name="blue"/>
+      <material name="red"/>
     </visual>
   </link>
